Commit message: Added simple maze and prepared for multi maze envs

File: urdfs/converter_input/generated/generated_maze_rov.urdf (robot description, URDF)
Before this commit: robot Labyrinth, 4 links, 3 joints
Links:
- link InnerDOFWalls: geometry visual mesh filename=meshes/generated_simple_maze_01.stl scale=0.001 0.001 0.001
