Commit message: fix: urdf and usds with better material properties and cleanup

File: urdfs/converter_input/real_maze_simple/real_maze_simple_01.urdf (robot description, URDF)
Before this commit: robot Labyrinth, 4 links, 3 joints
Links:
- link InnerDOFWalls: geometry visual mesh filename=meshes/InnerDOFWalls-Adjusted.STL scale=1 1 1
