Commit message: feat: Convexifying inner walls of hard maze

File: urdfs/converter_input/maze_no_holes/maze_no_holes.urdf (robot description, URDF)
Before this commit: robot Labyrinth, 5 links, 4 joints
Links:
- added link InnerDOFWallsCollisions; collision mesh filename=convex_walls/InnerDOFWalls_convex_1.STL scale=1 1 1; collision mesh filename=convex_walls/InnerDOFWalls_convex_10.STL scale=1 1 1
Joints:
- added joint FixedMazeWallCollisionsJoint: type fixed, parent InnerDOF, child InnerDOFWallsCollisions, origin xyz=0.0 0.0 0.0 rpy=0. 0. 0.
